File: Protoboard/PowerRails.kicad_sch (KiCad schematic)
At the start: 180 parts

Commit message: Protoboard Rev2 ready soon, needs checking
Parts:
- removed ? (x180): (no value), symbol Connector_Generic:Conn_01x01
