File: Protoboard/Prototype Board.kicad_sch (KiCad schematic)
At the start: 52 parts

Commit message: Improve Protoboard Rev2
Parts:
- added J215 (x120): Connectable_Pad_Group_01x04, Protoboard:Connectable_Pad_Group_01x04, symbol Prototype_Board:Connectable_Pad_Group_01x04
- added J216 (x12): ~, Protoboard:Connectable_Pad_Group_02x05, symbol Prototype_Board:Connectable_Pad_Group_02x05

Commit message: Protoboard Rev2 ready soon, needs checking
Parts:
- removed ?: (no value), symbol Device:LED
- removed ?: (no value), symbol ao_symbols:R
- added ?: (no value), symbol Device:LED
- added J170 (x32): Connectable_Pad_Group_01x02, Protoboard:Connectable_Pad_Group_01x02, symbol Prototype_Board:Connectable_Pad_Group_01x02
- added J347 (x3): Power_Rail_30, Protoboard:Power_Rail_30, symbol Prototype_Board:Power_Rail_30
- added R1: 4K7, symbol Device:R
- ?: symbol ao_symbols:CP -> Device:C_Polarized
- ? (x6): symbol Device:R_Potentiometer_MountingPin -> Device:R_Potentiometer
Connections:
- net +12V: now also J347.1, J347.1, J347.1, R1.2
- net GND: now also ?.1 (K), J347.2, J347.2, J347.2
- net 12V_Input: now reaches ?.1 (Pin_1), ?.1 (Pin_1), ?.2 (A), ?.2 (Pin_2), ?.2 (Pin_2), ?.3 (Pin_3), ?.3 (Pin_3)
- new net: ?.2 (A), R1.1
Other:
- removed sheet Power Rails
- note added: "A, B, C, D"
- note added: "Angled power headers in the back."
- note added: "Breadboard"
- note added: "Can mount either a pot, a 3mm pushbutton, or a 6mm one in those cursed frankensteined "footprints"."
- note added: "E, F, G, H"
- note added: "Flexible Inputs"
- note added: "I, J, K, L"
- note added: "I/O Pads"
- note added: "M, N, O, P"
- note added: "Power Input"
- note added: "Power Rail"
- note added: "[W], [X]"
- note added: "[Y], [Z]"
- note removed: "Angled power headers in the back, reverse polarityy protection"
- note removed: "Can mount either a pot, a 3mm pushbutton, or a 6mm one in those ultra-cursed frankensteined "footprints"."
- note removed: "Status indicator"
- note removed: "The breadboard pads and the I/O pads for pin headers at the edge of the board are not in the schematic because I couldn't figure out how to make KiCad place them on the PCB in a non-random order. Look it's my first real KiCad project I have zero idea what's up"
