File: Prototype Board/Prototype Board.kicad_pcb (KiCad board)
At the start: 2 copper layers, 99.1 x 99.1 mm, 224 parts, among them J1 Connectable_Pad_Group_01x02, J10 Connectable_Pad_Group_01x04, J100 Connectable_Pad_Group_01x04, J101 Connectable_Pad_Group_01x04, J102 Connectable_Pad_Group_01x04, J103 Connectable_Pad_Group_01x02, J104 Connectable_Pad_Group_01x04, J105 Connectable_Pad_Group_01x04, J106 Connectable_Pad_Group_01x04, J107 Connectable_Pad_Group_01x04, J108 Connectable_Pad_Group_01x04, J109 Connectable_Pad_Group_01x04, J11 Power_Rail_30, J110 Connectable_Pad_Group_01x04, J111 Connectable_Pad_Group_01x04, J112 Connectable_Pad_Group_01x02, J113 Connectable_Pad_Group_01x02, J114 Connectable_Pad_Group_01x04, J115 Connectable_Pad_Group_01x04, J116 Connectable_Pad_Group_01x04, J117 Connectable_Pad_Group_01x04, J120 Connectable_Pad_Group_01x04, J121 Connectable_Pad_Group_01x04, J122 Connectable_Pad_Group_01x04, J123 Connectable_Pad_Group_01x04, J124 Connectable_Pad_Group_01x02, J125 Connectable_Pad_Group_01x04, J126 Connectable_Pad_Group_01x04, J127 Connectable_Pad_Group_01x04, J128 Connectable_Pad_Group_01x04, J129 Connectable_Pad_Group_01x02, J13 Power_Rail_30, J130 Connectable_Pad_Group_01x04, J131 Connectable_Pad_Group_01x04, J132 Connectable_Pad_Group_01x04, J133 Connectable_Pad_Group_01x04, J134 Connectable_Pad_Group_01x02, J135 Connectable_Pad_Group_01x04, J136 Connectable_Pad_Group_01x04, J137 Connectable_Pad_Group_01x04, J138 Connectable_Pad_Group_01x04, J139 Connectable_Pad_Group_01x02, J140 Connectable_Pad_Group_01x04, J141 Connectable_Pad_Group_01x04, J142 Connectable_Pad_Group_01x04, J143 Connectable_Pad_Group_01x04, J146 Connectable_Pad_Group_01x02, J147 Connectable_Pad_Group_01x04, J148 Connectable_Pad_Group_01x04, J149 Connectable_Pad_Group_01x04, J15 Power_Rail_30, J150 Connectable_Pad_Group_01x04, J151 Connectable_Pad_Group_01x02, J152 Connectable_Pad_Group_01x02, J153 Connectable_Pad_Group_01x02, J154 Connectable_Pad_Group_01x02, J155 Connectable_Pad_Group_01x04, J156 Connectable_Pad_Group_01x04, J157 Connectable_Pad_Group_01x04, J158 Connectable_Pad_Group_01x04, J159 Connectable_Pad_Group_01x02, J16 Connectable_Pad_Group_01x02, J160 Connectable_Pad_Group_01x04, J161 Connectable_Pad_Group_01x04, J162 Connectable_Pad_Group_01x04, J163 Connectable_Pad_Group_01x04, J164 Connectable_Pad_Group_01x04, J165 Connectable_Pad_Group_01x04, J166 Connectable_Pad_Group_01x04, J167 Connectable_Pad_Group_01x04, J17 Connectable_Pad_Group_01x04, J174 Conn_01x03_Male, J175 Conn_01x03_Male, J176 Conn_01x01, J177 Conn_01x01, J178 Conn_01x01, J179 Conn_01x01, J18 Connectable_Pad_Group_01x04, J180 Conn_01x01, J181 Conn_01x01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

Commit message: Standardize prototype board folder name, Rev 2B
Other:
- board text added: "Perma Proto for Synth Array Rev 02b - Aria Salvatrice"
- board text removed: "Perma Proto for Synth Array Rev 02 - Aria Salvatrice"
Changed lines of the file:
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@@
   (title_block
     (title "Perma Proto for Synth Array")
-    (date "2022-08-27")
-    (rev "02")
+    (date "2022-10-04")
+    (rev "02b")
     (company "Aria Salvatrice")
   )
@@
     (effects (font (size 1 1) (thickness 0.15)) (justify mirror))
   )
-  (gr_text "JLCJLCJLCJLC" (at 186.69 62.23 90) (layer "B.SilkS")
-    (effects (font (size 1 1) (thickness 0.15)) (justify left mirror))
-  )
   (gr_text "+" (at 180.34 73.66) (layer "B.SilkS")
     (effects (font (size 1 1) (thickness 0.15)) (justify mirror))
@@
     (effects (font (size 1 1) (thickness 0.15)) (justify mirror))
   )
-  (gr_text "Perma Proto for Synth Array\nRev 02 - Aria Salvatrice" (at 184.15 62.23 90) (layer "B.SilkS")
+  (gr_text "Perma Proto for Synth Array\nRev 02b - Aria Salvatrice" (at 184.15 62.23 90) (layer "B.SilkS")
     (effects (font (size 1 1) (thickness 0.15)) (justify left mirror))
   )
@@
     (effects (font (size 1 1) (thickness 0.15)))
   )
+  (gr_text "JLCJLCJLCJLC" (at 186.69 62.23 90) (layer "Cmts.User")
+    (effects (font (size 1 1) (thickness 0.15)) (justify left mirror))
+  )
   (gr_text "TODO LIST\n- Imported symbol to replace\n- Pass DRC (already pass the important parts)" (at 205.74 55.88) (layer "Cmts.User")
     (effects (font (size 1 1) (thickness 0.15)) (justify left))
@@
   (segment (start 144.78 117.775) (end 145.04 118.035) (width 1) (layer "F.Cu") (net 191))
   (segment (start 162.85 117.715) (end 162.53 118.035) (width 1) (layer "F.Cu") (net 192))
-  (segment (start 161.53 123.535) (end 162.53 124.535) (width 1) (layer "F.Cu") (net 192))
-  (segment (start 162.85 111.76) (end 162.85 117.715) (width 1) (layer "F.Cu") (net 192))
-  (segment (start 162.53 118.035) (end 161.53 119.035) (width 1) (layer "F.Cu") (net 192))
-  (segment (start 162.53 124.535) (end 162.53 126.68) (width 1) (layer "F.Cu") (net 192))
-  (segment (start 161.53 119.035) (end 161.53 123.535) (width 1) (layer "F.Cu") (net 192))
+  (segment (start 161.2146 123.535) (end 162.2146 124.535) (width 1) (layer "F.Cu") (net 192))
+  (segment (start 162.5346 111.76) (end 162.5346 117.715) (width 1) (layer "F.Cu") (net 192))
+  (segment (start 162.2146 118.035) (end 161.2146 119.035) (width 1) (layer "F.Cu") (net 192))
+  (segment (start 162.2146 124.535) (end 162.2146 126.68) (width 1) (layer "F.Cu") (net 192))
+  (segment (start 161.2146 119.035) (end 161.2146 123.535) (width 1) (layer "F.Cu") (net 192))
   (segment (start 162.53 126.68) (end 162.85 127) (width 1) (layer "F.Cu") (net 192))
-  (segment (start 158.03 118.035) (end 159.03 119.035) (width 1) (layer "F.Cu") (net 193))
-  (segment (start 157.77 111.76) (end 157.77 117.775) (width 1) (layer "F.Cu") (net 193))
-  (segment (start 159.03 119.035) (end 159.03 123.535) (width 1) (layer "F.Cu") (net 193))
+  (segment (start 157.7146 118.035) (end 158.7146 119.035) (width 1) (layer "F.Cu") (net 193))
+  (segment (start 157.4546 111.76) (end 157.4546 117.775) (width 1) (layer "F.Cu") (net 193))
+  (segment (start 158.7146 119.035) (end 158.7146 123.535) (width 1) (layer "F.Cu") (net 193))
   (segment (start 158.03 126.74) (end 157.77 127) (width 1) (layer "F.Cu") (net 193))
-  (segment (start 158.03 124.535) (end 158.03 126.74) (width 1) (layer "F.Cu") (net 193))
-  (segment (start 159.03 123.535) (end 158.03 124.535) (width 1) (layer "F.Cu") (net 193))
+  (segment (start 157.7146 124.535) (end 157.7146 126.74) (width 1) (layer "F.Cu") (net 193))
+  (segment (start 158.7146 123.535) (end 157.7146 124.535) (width 1) (layer "F.Cu") (net 193))
   (segment (start 157.77 117.775) (end 158.03 118.035) (width 1) (layer "F.Cu") (net 193))
   (segment (start 175.26 124.245) (end 174.97 124.535) (width 0.25) (layer "F.Cu") (net 194))
@@
   (segment (start 147.32 114.27) (end 147.29 114.3) (width 1) (layer "F.Cu") (net 196))
   (segment (start 147.32 111.76) (end 147.32 114.27) (width 1) (layer "F.Cu") (net 196))
-  (segment (start 160.31 111.76) (end 160.31 114.27) (width 1) (layer "F.Cu") (net 197))
+  (segment (start 159.9946 111.76) (end 159.9946 114.27) (width 1) (layer "F.Cu") (net 197))
   (segment (start 160.31 114.27) (end 160.28 114.3) (width 1) (layer "F.Cu") (net 197))
   (segment (start 172.72 111.76) (end 172.72 114.27) (width 1) (layer "F.Cu") (net 198))
